File: Hardware/RN-52 Breakout.brd (EAGLE design)
At the start: 35.6 x 51.1 mm, 13 parts, among them U1 BLUETOOTH-RN-52

Commit message: Added Version
Added Version and cleaned up repo
Other:
- board text added: "V10"
Changed lines of the file:
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@@
 <layer number="106" name="bPlate" color="7" fill="1" visible="no" active="yes"/>
 <layer number="107" name="Crop" color="7" fill="1" visible="no" active="yes"/>
-<layer number="108" name="tplace-old" color="10" fill="1" visible="yes" active="yes"/>
-<layer number="109" name="ref-old" color="11" fill="1" visible="yes" active="yes"/>
+<layer number="108" name="tplace-old" color="10" fill="1" visible="no" active="yes"/>
+<layer number="109" name="ref-old" color="11" fill="1" visible="no" active="yes"/>
 <layer number="116" name="Patch_BOT" color="9" fill="4" visible="no" active="yes"/>
 <layer number="121" name="_tsilk" color="7" fill="1" visible="no" active="yes"/>
@@
 <text x="32.512" y="3.175" size="1.27" layer="22" font="vector" ratio="15" rot="MR0">PCM_CK</text>
 <text x="32.512" y="0.635" size="1.27" layer="22" font="vector" ratio="15" rot="MR0">GND</text>
+<text x="20.32" y="48.26" size="1.778" layer="16" font="vector" ratio="15" rot="MR0">V10</text>
 </plain>
 <attributes>
